Commit message: changed jetank namespace
changed URDF , Description , controllers and bridge configuration

File: urdf/jetank_controllers.xacro (robot description, xacro)
@@ -16,4 +16,6 @@
 		position or velocity
 	-->
+	<!-- gz_ros2_control runs the controller_manager for you however this can come with some issues later when trying to remap -->
+	<!-- https://robotics.stackexchange.com/questions/103767/class-gazebo-ros2-control-gazebosystem-with-base-class-type-hardware-interface -->
 	<ros2_control name="jetank_controller" type="system">
 		<hardware>

File: urdf/jetank_joints.xacro (robot description, xacro)
@@ -15,4 +15,63 @@
     </xacro:macro>
     <!-- ================ JOINTS ================ -->
+    <!-- SERVO's -->
+    <xacro:joint joint_name="turn_ARM" parent_name="BEARING" child_name="ARM_LOWER" joint_type="revolute">
+        <origin xyz="0 0.0002 -0.0080" rpy="${PI} 0 0" />
+        <axis xyz="0 -0.0021 1" />
+        <limit lower="-${PI/2}" upper="${PI/2}" effort="1000000" velocity="1000000" />
+    </xacro:joint>
+    <xacro:joint joint_name="SERVO_UPPER_" parent_name="ARM_MIDDLE" child_name="SERVO_UPPER" joint_type="revolute">
+        <origin xyz="-0.0672 0.0672 0" rpy="${PI/2} 0 0" />
+        <axis xyz="-0.0036 1 0.0021" />
+        <limit lower="-2" upper="1" effort="1000000" velocity="1000000" />
+    </xacro:joint>
+    <xacro:joint joint_name="SERVO_LOWER_" parent_name="SERVO_LOWER" child_name="ARM_MIDDLE" joint_type="revolute">
+        <origin xyz="-0.0271 0 0.0184" rpy="0 0 0" />
+        <axis xyz="-0.0036 -0.0021 1" />
+        <limit lower="0" upper="${PI/4}" effort="1000000" velocity="1000000" />
+    </xacro:joint>
+    <!-- WHEELS -->
+    <xacro:joint joint_name="DRIVING_WHEEL_RIGHT" parent_name="base_link" child_name="DRIVER_WHEEL_R" joint_type="continuous">
+        <origin xyz="0.0560 0.0442 0.0133" rpy="-${PI/2} 0 -${PI}" />
+        <axis xyz="0.0036 0.0021 -1" />
+        <limit/>
+    </xacro:joint>
+    <xacro:joint joint_name="DRIVING_WHEEL_LEFT" parent_name="base_link" child_name="DRIVER_WHEEL_L" joint_type="continuous">
+        <origin xyz="-0.0625 -0.0442 0.0133" rpy="${PI/2} 0 ${PI}" />
+        <axis xyz="-0.0036 0.0021 1" />
+        <limit/>
+    </xacro:joint>
+        <xacro:joint joint_name="FREE_WHEEL_LEFT" parent_name="base_link" child_name="FREE_WHEEL_L" joint_type="continuous">
+        <origin xyz="0.0560 -0.0442 0.0133" rpy="${PI/2} 0 -${PI}" />
+        <axis xyz="-0.0036 0.0021 1" />
+        <limit/>
+    </xacro:joint>
+    <xacro:joint joint_name="FREE_WHEEL_RIGHT" parent_name="base_link" child_name="FREE_WHEEL_R" joint_type="continuous">
+        <origin xyz="-0.0625 0.0442 0.0133" rpy="-${PI/2} 0 -${PI}" />
+        <axis xyz="0.0036 0.0021 -1" />
+        <limit/>
+    </xacro:joint>
+    <!-- GRIPPER -->
+    <xacro:joint joint_name="GRIPPER_RIGHT_2" parent_name="GRIPPER_R1" child_name="GRIPPER_R2" joint_type="revolute">
+        <origin xyz="-0.025 0 -0.0155" rpy="${PI} -${PI/4 - 0.09} 0" />
+        <axis xyz="-0.3503 -0.0032 0.9366" />
+        <limit lower="0" upper="${PI/4}" effort="1000000" velocity="1000000" />
+    </xacro:joint>
+    <xacro:joint joint_name="GRIPPER_LEFT_2" parent_name="GRIPPER_L1" child_name="GRIPPER_L2" joint_type="revolute">
+        <origin xyz="-0.025 0 -0.0155" rpy="0 -${PI/4 - 0.09} 0" />
+        <axis xyz="0.3503 0.0032 0.9366" />
+        <limit lower="0" upper="${PI/4}" effort="1000000" velocity="1000000" />
+    </xacro:joint>
+    <xacro:joint joint_name="GRIPPER_RIGHT_1" parent_name="GRIPPER_BASE" child_name="GRIPPER_R1" joint_type="revolute">
+        <origin xyz="0.0419 0.0051 -0.0149" rpy="0 -0.0169 ${PI}" />
+        <axis xyz="-0.3503 -0.0032 0.9366" />
+        <limit lower="0" upper="${PI/4}" effort="1000000" velocity="1000000" />
+    </xacro:joint>
+    <xacro:joint joint_name="GRIPPER_LEFT_1" parent_name="GRIPPER_BASE" child_name="GRIPPER_L1" joint_type="revolute">
+        <origin xyz="0.0420 -0.0049 -0.0149" rpy="0 -0.0169 ${PI}" />
+        <axis xyz="0.3503 0.0032 -0.9366" />
+        <limit lower="0" upper="${PI/4}" effort="1000000" velocity="1000000" />
+    </xacro:joint>
+    <!-- fixed joints -->
     <xacro:joint joint_name="base_link_rigid_ANTENNA_L_BASE_JOINT" parent_name="base_link" child_name="ANTENNA_L" joint_type="fixed">
         <origin xyz="0.0718 -0.0442 0.0576" rpy="${PI/2} 0 -${PI}" />
@@ -30,19 +89,4 @@
         <limit/>
     </xacro:joint>
-    <xacro:joint joint_name="turn_ARM" parent_name="BEARING" child_name="ARM_LOWER" joint_type="revolute">
-        <origin xyz="0 0.0002 -0.0080" rpy="${PI} 0 0" />
-        <axis xyz="0 -0.0021 1" />
-        <limit lower="-${PI/2}" upper="${PI/2}" effort="1000000" velocity="1000000" />
-    </xacro:joint>
-    <xacro:joint joint_name="FREE_WHEEL_LEFT" parent_name="base_link" child_name="FREE_WHEEL_L" joint_type="continuous">
-        <origin xyz="0.0560 -0.0442 0.0133" rpy="${PI/2} 0 -${PI}" />
-        <axis xyz="-0.0036 0.0021 1" />
-        <limit/>
-    </xacro:joint>
-    <xacro:joint joint_name="FREE_WHEEL_RIGHT" parent_name="base_link" child_name="FREE_WHEEL_R" joint_type="continuous">
-        <origin xyz="-0.0625 0.0442 0.0133" rpy="-${PI/2} 0 -${PI}" />
-        <axis xyz="0.0036 0.0021 -1" />
-        <limit/>
-    </xacro:joint>
     <xacro:joint joint_name="CAM_HOLDER_rigid_CAMERA_CAMERA_HOLDER" parent_name="CAM_HOLDER" child_name="CAMERA" joint_type="fixed">
         <origin xyz="-0.0338 0 -0.0001" rpy="${PI/2} 0 0" />
@@ -55,48 +99,8 @@
         <limit/>
     </xacro:joint>
-    <xacro:joint joint_name="GRIPPER_LEFT_1" parent_name="GRIPPER_BASE" child_name="GRIPPER_L1" joint_type="revolute">
-        <origin xyz="0.0419 0.0051 -0.0149" rpy="0 -0.0169 ${PI}" />
-        <axis xyz="0.3503 0.0032 -0.9366" />
-        <limit lower="-${PI/4}" upper="0.0" effort="1000000" velocity="1000000" />
-    </xacro:joint>
-    <xacro:joint joint_name="GRIPPER_LEFT_2" parent_name="GRIPPER_L1" child_name="GRIPPER_L2" joint_type="revolute">
-        <origin xyz="-0.0281 0 -0.0104" rpy="${PI} 0 0" />
-        <axis xyz="-0.3503 0.0032 -0.9366" />
-        <limit lower="-${PI/4}" upper="0.0" effort="1000000" velocity="1000000" />
-    </xacro:joint>
-    <xacro:joint joint_name="SERVO_UPPER_" parent_name="ARM_MIDDLE" child_name="SERVO_UPPER" joint_type="revolute">
-        <origin xyz="-0.0672 0.0672 0" rpy="${PI/2} 0 0" />
-        <axis xyz="-0.0036 1 0.0021" />
-        <limit lower="-2" upper="1" effort="1000000" velocity="1000000" />
-    </xacro:joint>
-    <xacro:joint joint_name="SERVO_LOWER_" parent_name="SERVO_LOWER" child_name="ARM_MIDDLE" joint_type="revolute">
-        <origin xyz="-0.0271 0 0.0184" rpy="0 0 0" />
-        <axis xyz="-0.0036 -0.0021 1" />
-        <limit lower="0" upper="${PI/4}" effort="1000000" velocity="1000000" />
-    </xacro:joint>
     <xacro:joint joint_name="ARM_LOWER_Rigid_SERVO_LOWER_ARM_LOWER" parent_name="ARM_LOWER" child_name="SERVO_LOWER" joint_type="fixed">
         <origin xyz="0.0135 0.0200 0.0672" rpy="${PI/2} 0 0" />
         <axis/>
         <limit/>
-    </xacro:joint>
-    <xacro:joint joint_name="DRIVING_WHEEL_RIGHT" parent_name="base_link" child_name="DRIVER_WHEEL_R" joint_type="continuous">
-        <origin xyz="0.0560 0.0442 0.0133" rpy="-${PI/2} 0 -${PI}" />
-        <axis xyz="0.0036 0.0021 -1" />
-        <limit/>
-    </xacro:joint>
-    <xacro:joint joint_name="DRIVING_WHEEL_LEFT" parent_name="base_link" child_name="DRIVER_WHEEL_L" joint_type="continuous">
-        <origin xyz="-0.0625 -0.0442 0.0133" rpy="${PI/2} 0 ${PI}" />
-        <axis xyz="-0.0036 0.0021 1" />
-        <limit/>
-    </xacro:joint>
-    <xacro:joint joint_name="GRIPPER_RIGHT_2" parent_name="GRIPPER_R1" child_name="GRIPPER_R2" joint_type="revolute">
-        <origin xyz="-0.0281 0 -0.0105" rpy="0 0 0" />
-        <axis xyz="0.3503 0.0032 -0.9366" />
-        <limit lower="-${PI/4}" upper="0" effort="1000000" velocity="1000000" />
-    </xacro:joint>
-    <xacro:joint joint_name="GRIPPER_RIGHT_1" parent_name="GRIPPER_BASE" child_name="GRIPPER_R1" joint_type="revolute">
-        <origin xyz="0.0420 -0.0049 -0.0149" rpy="0 -0.0169 ${PI}" />
-        <axis xyz="0.3503 0.0032 -0.9366" />
-        <limit lower="0" upper="${PI/4}" effort="1000000" velocity="1000000" />
     </xacro:joint>
     <xacro:joint joint_name="ARM_UPPER_rigid_GRIPPER_BASE_ARM_UPPER" parent_name="ARM_UPPER" child_name="GRIPPER_BASE" joint_type="fixed">

Commit message: changed Jetank controllers and urdf files for compatability with Gazebo ignition and ROS Humble

File: urdf/jetank_controllers.xacro (robot description, xacro)
@@ -1,15 +1,15 @@
 <?xml version="1.0"?>
 <robot xmlns:xacro="http://www.ros.org/wiki/xacro" name="jetank">
-    	<!-- other of kinds of systems are 'actuator' and 'sensor' but 'system' is more general -->
+	<!-- other of kinds of systems are 'actuator' and 'sensor' but 'system' is more general -->
 	<!--
-		inside the ros2_control tag we define a plugin inside the <hardware> tag to say
+		inside the ros2_control tag we define a plugin inside the hardware tag to say
 		which plugins to load in Gazebo to simulate a real hardware interface
 		further we need to define the joints that are controllable.
-		In our case we have:
-		- the wheels of the Jetank
-		- the base of the arm
-		- the 2 servo's
-		- the gripper
-		- (perhaps the camera holder)
+		In our case we have
+		 	the wheels of the Jetank
+		 	the base of the arm
+		 	the 2 servos
+		 	the gripper
+		 	perhaps the camera holder
 		each joint will have state_interfaces
 		and command intefaces. That being either
@@ -20,5 +20,5 @@
 	<ros2_control name="jetank_controller" type="system">
 		<hardware>
-			<plugin>gz_ros2_control/GazeboSimSystem</plugin>
+			<plugin>ign_ros2_control/IgnitionSystem</plugin>
 		</hardware>
 		<joint name="turn_ARM">

File: urdf/jetank_joints.xacro (robot description, xacro)
@@ -19,15 +19,15 @@
         <origin xyz="0 0.0002 -0.0080" rpy="${PI} 0 0" />
         <axis xyz="0 -0.0021 1" />
-        <limit lower="-${PI/2}" upper="${PI/2}" effort="1000000" velocity="1000000" />
+        <limit lower="-${PI/2}" upper="${PI/2}" effort="50" velocity="10" />
     </xacro:joint>
     <xacro:joint joint_name="SERVO_UPPER_" parent_name="ARM_MIDDLE" child_name="SERVO_UPPER" joint_type="revolute">
         <origin xyz="-0.0672 0.0672 0" rpy="${PI/2} 0 0" />
         <axis xyz="-0.0036 1 0.0021" />
-        <limit lower="-2" upper="1" effort="1000000" velocity="1000000" />
+        <limit lower="-2" upper="1" effort="50" velocity="10" />
     </xacro:joint>
     <xacro:joint joint_name="SERVO_LOWER_" parent_name="SERVO_LOWER" child_name="ARM_MIDDLE" joint_type="revolute">
         <origin xyz="-0.0271 0 0.0184" rpy="0 0 0" />
         <axis xyz="-0.0036 -0.0021 1" />
-        <limit lower="0" upper="${PI/4}" effort="1000000" velocity="1000000" />
+        <limit lower="0" upper="${PI/4}" effort="50" velocity="10" />
     </xacro:joint>
     <!-- WHEELS -->
@@ -56,20 +56,20 @@
         <origin xyz="-0.025 0 -0.0155" rpy="${PI} -${PI/4 - 0.09} 0" />
         <axis xyz="-0.3503 -0.0032 0.9366" />
-        <limit lower="0" upper="${PI/4}" effort="1000000" velocity="1000000" />
+        <limit lower="0" upper="${PI/4}" effort="75" velocity="10" />
     </xacro:joint>
     <xacro:joint joint_name="GRIPPER_LEFT_2" parent_name="GRIPPER_L1" child_name="GRIPPER_L2" joint_type="revolute">
         <origin xyz="-0.025 0 -0.0155" rpy="0 -${PI/4 - 0.09} 0" />
         <axis xyz="0.3503 0.0032 0.9366" />
-        <limit lower="0" upper="${PI/4}" effort="1000000" velocity="1000000" />
+        <limit lower="0" upper="${PI/4}" effort="75" velocity="10" />
     </xacro:joint>
     <xacro:joint joint_name="GRIPPER_RIGHT_1" parent_name="GRIPPER_BASE" child_name="GRIPPER_R1" joint_type="revolute">
         <origin xyz="0.0419 0.0051 -0.0149" rpy="0 -0.0169 ${PI}" />
         <axis xyz="-0.3503 -0.0032 0.9366" />
-        <limit lower="0" upper="${PI/4}" effort="1000000" velocity="1000000" />
+        <limit lower="0" upper="${PI/4}" effort="75" velocity="10" />
     </xacro:joint>
     <xacro:joint joint_name="GRIPPER_LEFT_1" parent_name="GRIPPER_BASE" child_name="GRIPPER_L1" joint_type="revolute">
         <origin xyz="0.0420 -0.0049 -0.0149" rpy="0 -0.0169 ${PI}" />
         <axis xyz="0.3503 0.0032 -0.9366" />
-        <limit lower="0" upper="${PI/4}" effort="1000000" velocity="1000000" />
+        <limit lower="0" upper="${PI/4}" effort="75" velocity="10" />
     </xacro:joint>
     <!-- fixed joints -->

File: urdf/jetank_sensors.xacro (robot description, xacro)
@@ -39,10 +39,7 @@
 		</sensor>
 	</gazebo>
-	<!--
-		required for Gazebo such that ros2_control can work.
-		We need to load a config file to tell what controllers to load
-	-->
+	<!-- required for Gazebo such that ros2_control can work. We need to load a config file to tell what controllers to load -->
 	<gazebo>
-		<plugin filename="gz_ros2_control-system" name="gz_ros2_control::GazeboSimROS2ControlPlugin">
+		<plugin filename="ign_ros2_control-system" name="ign_ros2_control::IgnitionROS2ControlPlugin">
 			<parameters>
 				$(find jetank_description)/config/jetank_controllers.yaml
